File: hw/adapter_soldered/fpga_wide/adapter_soldered.kicad_pcb (KiCad board)
At the start: 2 copper layers, 4.9 x 17.8 mm, 13 parts, among them J1 1-2328702-0, Q1 2DC4617QLP, U1 SPI Flash, U3 NCP171AMX165160TCG

Commit message: hw/ - DFM/manufacturability improvements for FPGA flex PCB variant. New extra-wide adapter_soldered/breakout_wson for WSON 8x6.
Parts:
- U2: footprint flashkeeper:FlashkeeperFPGASoM -> flashkeeper:FlashkeeperFPGASoM_ReducedPins
- moved JP1 5.28 mm to (149.1, 106.8), turned to 180 degrees
- moved R2 1.71 mm to (143.5, 118.9), turned to -90 degrees
- moved Q1 1.36 mm to (143.8, 117.3)
- moved D2 0.15 mm to (145.1, 118.9)
- moved R1 0.10 mm to (145.0, 118.2)
- moved C1 0.05 mm to (145.0, 116.8)
- moved D1 0.05 mm to (145.1, 117.5)
- turned U3 to 90 degrees
Connections:
- U3 pad 3: VCC -> +2V5
- U3 pad 4: VCC -> +2V5
Routing:
- net VCC: track 28.1 -> 10.1 mm, vias 2 -> 1
- net +2V5: track 17.8 -> 21.8 mm
- net Net-(D1-A): track 5.18 -> 1.85 mm
- net CDONE: track 19.5 -> 17.7 mm
- net DRX: track 6.69 -> 5.60 mm
- net Net-(Q1-B): track 2.05 -> 0.98 mm
- net Net-(D2-A): track 4.10 -> 4.72 mm
- net DTX: track 4.69 -> 5.29 mm
- net GND: track 8.29 -> 8.85 mm, vias 3 -> 5
- net Net-(BT1-+): track 22.2 -> 22.7 mm
Other:
- board size 4.9 x 17.8 mm -> 4.9 x 17.9 mm
