File: hw/adapter_soldered/fpga_wide/adapter_soldered.kicad_sch (KiCad schematic)
At the start: 13 parts, among them J1 1-2328702-0, Q1 2DC4617QLP, U1 SPI Flash, U3 NCP171AMX165160TCG

Commit message: hw/ - DFM/manufacturability improvements for FPGA flex PCB variant. New extra-wide adapter_soldered/breakout_wson for WSON 8x6.
Parts:
- U1: footprint flashkeeper:SolderConnector_SOIC8Wide -> flashkeeper:SolderConnector_SOIC8Wide_1.5mmLift
- U2: footprint flashkeeper:FlashkeeperFPGASoM -> flashkeeper:FlashkeeperFPGASoM_ReducedPins
Connections:
- net +2V5: now also U3.3 (IN), U3.4 (ENA)
- net VCC: no longer U3.3 (IN), U3.4 (ENA)
Changed lines of the file:
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@@
 			)
 		)
-		(property "Footprint" "flashkeeper:SolderConnector_SOIC8Wide"
+		(property "Footprint" "flashkeeper:SolderConnector_SOIC8Wide_1.5mmLift"
 			(at 236.22 101.6 0)
 			(hide yes)
@@
 			)
 		)
-		(property "Footprint" "flashkeeper:FlashkeeperFPGASoM"
+		(property "Footprint" "flashkeeper:FlashkeeperFPGASoM_ReducedPins"
 			(at 179.07 101.6 0)
 			(hide yes)
@@
 	)
 	(symbol
-		(lib_id "power:VCC")
+		(lib_id "power:+2V5")
 		(at 92.71 78.74 0)
 		(unit 1)
@@
 		(in_pos_files yes)
 		(dnp no)
-		(fields_autoplaced yes)
-		(property "Reference" "#PWR010"
+		(property "Reference" "#PWR014"
 			(at 92.71 82.55 0)
 			(hide yes)
@@
 			)
 		)
-		(property "Value" "VCC"
-			(at 92.71 74.6069 0)
+		(property "Value" "+2V5"
+			(at 92.71 74.676 0)
 			(show_name no)
 			(do_not_autoplace no)
@@
 			)
 		)
-		(property "Description" "Power symbol creates a global label with name \"VCC\""
+		(property "Description" "Power symbol creates a global label with name \"+2V5\""
 			(at 92.71 78.74 0)
 			(hide yes)
@@
 			(project "adapter_soldered"
 				(path "/44cdec2e-7ad1-4d15-a8ec-478a4c576cd0"
-					(reference "#PWR010")
-					(unit 1)
-				)
+					(reference "#PWR014")
+					(unit 1)
+				)
